File: PB170/PB170.sch (KiCad schematic (older format))
At the start: 33 parts, among them J1 USB_C_Receptacle_USB2.0-Conne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, J2 USB_B_Micro, Q1 P-MOSFET-MLP_HS, Q2 BC817, SW1 SW_MEC_5E, SW2 SW_MEC_5E

Commit message: Setup xor component, create ALU and ADDER sheets
Changed lines of the file:
@@
 $Descr A4 11693 8268
 encoding utf-8
-Sheet 1 3
+Sheet 1 5
 Title ""
 Date ""
@@
 F1 "newParts.sch" 50
 $EndSheet
+$Sheet
+S 8750 1300 900  1450
+U 600A4AF3
+F0 "SheetALU" 50
+F1 "alu.sch" 50
+$EndSheet
 $EndSCHEMATC
