File: PB170/alu.sch (KiCad schematic (older format))
At the start: 0 parts

Commit message: Create adder
Changed lines of the file:
@@
 F0 "SheetAdder" 50
 F1 "adder.sch" 50
+F2 "IN_A0" I L 3650 1800 50
+F3 "IN_A1" I L 3650 1900 50
+F4 "IN_A2" I L 3650 2000 50
+F5 "IN_A3" I L 3650 2100 50
+F6 "IN_SUB" I L 3650 2450 50
+F7 "IN_B0" I L 3650 2700 50
+F8 "IN_B1" I L 3650 2800 50
+F9 "IN_B2" I L 3650 2900 50
+F10 "IN_B3" I L 3650 3000 50
+F11 "OUT_Y0" O R 4900 2100 50
+F12 "OUT_Y1" O R 4900 2200 50
+F13 "OUT_Y2" O R 4900 2300 50
+F14 "OUT_Y3" O R 4900 2400 50
+F15 "COUT_3" O R 4900 2800 50
+F16 "COUT_2" O R 4900 2700 50
 $EndSheet
 $EndSCHEMATC
