File: PB170/newParts.sch (KiCad schematic (older format))
At the start: 9 parts, among them U2 74HC08, U3 74HC4511D, U4 HEF4518BT, U5 74HC32

Commit message: Add alu output flags
Parts:
- added U? (x5): 74HC00, Package_SO:TSSOP-14_4.4x5mm_P0.65mm, symbol 74xx:74HC00
Changed lines of the file:
@@
-$EndComp
-$Comp
-L 74xx:74HC86 U?
-U 1 1 600A8380
-P 1400 4200
-F 0 "U?" H 1400 4525 50  0000 C CNN
-F 1 "74HC86" H 1400 4434 50  0000 C CNN
-F 2 "Package_SO:TSSOP-14_4.4x5mm_P0.65mm" H 1400 4200 50  0001 C CNN
-F 3 "https://datasheet.lcsc.com/szlcsc/Texas-Instruments-TI-SN74AHC86PWR_C117522.pdf" H 1400 4200 50  0001 C CNN
-F 4 "C117522" H 1400 4200 50  0001 C CNN "LCSC"
-	1    1400 4200
-	1    0    0    -1
-$EndComp
-$Comp
-L 74xx:74HC86 U?
-U 2 1 600AA188
-P 2200 4200
-F 0 "U?" H 2200 4525 50  0000 C CNN
-F 1 "74HC86" H 2200 4434 50  0000 C CNN
-F 2 "Package_SO:TSSOP-14_4.4x5mm_P0.65mm" H 2200 4200 50  0001 C CNN
-F 3 "https://datasheet.lcsc.com/szlcsc/Texas-Instruments-TI-SN74AHC86PWR_C117522.pdf" H 2200 4200 50  0001 C CNN
-F 4 "C117522" H 2200 4200 50  0001 C CNN "LCSC"
-	2    2200 4200
-	1    0    0    -1
-$EndComp
-$Comp
-L 74xx:74HC86 U?
-U 3 1 600AF551
-P 3000 4200
-F 0 "U?" H 3000 4525 50  0000 C CNN
-F 1 "74HC86" H 3000 4434 50  0000 C CNN
-F 2 "Package_SO:TSSOP-14_4.4x5mm_P0.65mm" H 3000 4200 50  0001 C CNN
-F 3 "https://datasheet.lcsc.com/szlcsc/Texas-Instruments-TI-SN74AHC86PWR_C117522.pdf" H 3000 4200 50  0001 C CNN
-F 4 "C117522" H 3000 4200 50  0001 C CNN "LCSC"
-	3    3000 4200
-	1    0    0    -1
-$EndComp
-$Comp
-L 74xx:74HC86 U?
-U 4 1 600B0ABE
-P 3800 4200
-F 0 "U?" H 3800 4525 50  0000 C CNN
-F 1 "74HC86" H 3800 4434 50  0000 C CNN
-F 2 "Package_SO:TSSOP-14_4.4x5mm_P0.65mm" H 3800 4200 50  0001 C CNN
-F 3 "https://datasheet.lcsc.com/szlcsc/Texas-Instruments-TI-SN74AHC86PWR_C117522.pdf" H 3800 4200 50  0001 C CNN
-F 4 "C117522" H 3800 4200 50  0001 C CNN "LCSC"
-	4    3800 4200
-	1    0    0    -1
 $EndComp
 $Comp
@@
 $Comp
 L 74xx:74HC86 U?
+U 4 1 600B0ABE
+P 3800 4200
+F 0 "U?" H 3800 4525 50  0000 C CNN
+F 1 "74HC86" H 3800 4434 50  0000 C CNN
+F 2 "Package_SO:TSSOP-14_4.4x5mm_P0.65mm" H 3800 4200 50  0001 C CNN
+F 3 "https://datasheet.lcsc.com/szlcsc/Texas-Instruments-TI-SN74AHC86PWR_C117522.pdf" H 3800 4200 50  0001 C CNN
+F 4 "C117522" H 3800 4200 50  0001 C CNN "LCSC"
+	4    3800 4200
+	1    0    0    -1
+$EndComp
+$Comp
+L 74xx:74HC86 U?
+U 1 1 600A8380
+P 1400 4200
+F 0 "U?" H 1400 4525 50  0000 C CNN
+F 1 "74HC86" H 1400 4434 50  0000 C CNN
+F 2 "Package_SO:TSSOP-14_4.4x5mm_P0.65mm" H 1400 4200 50  0001 C CNN
+F 3 "https://datasheet.lcsc.com/szlcsc/Texas-Instruments-TI-SN74AHC86PWR_C117522.pdf" H 1400 4200 50  0001 C CNN
+F 4 "C117522" H 1400 4200 50  0001 C CNN "LCSC"
+	1    1400 4200
+	1    0    0    -1
+$EndComp
+$Comp
+L 74xx:74HC86 U?
+U 3 1 600AF551
+P 3000 4200
+F 0 "U?" H 3000 4525 50  0000 C CNN
+F 1 "74HC86" H 3000 4434 50  0000 C CNN
+F 2 "Package_SO:TSSOP-14_4.4x5mm_P0.65mm" H 3000 4200 50  0001 C CNN
+F 3 "https://datasheet.lcsc.com/szlcsc/Texas-Instruments-TI-SN74AHC86PWR_C117522.pdf" H 3000 4200 50  0001 C CNN
+F 4 "C117522" H 3000 4200 50  0001 C CNN "LCSC"
+	3    3000 4200
+	1    0    0    -1
+$EndComp
+$Comp
+L 74xx:74HC86 U?
 U 5 1 600B2251
 P 4550 4200
@@
 	1    0    0    -1
 $EndComp
+$Comp
+L 74xx:74HC86 U?
+U 2 1 600AA188
+P 2200 4200
+F 0 "U?" H 2200 4525 50  0000 C CNN
+F 1 "74HC86" H 2200 4434 50  0000 C CNN
+F 2 "Package_SO:TSSOP-14_4.4x5mm_P0.65mm" H 2200 4200 50  0001 C CNN
+F 3 "https://datasheet.lcsc.com/szlcsc/Texas-Instruments-TI-SN74AHC86PWR_C117522.pdf" H 2200 4200 50  0001 C CNN
+F 4 "C117522" H 2200 4200 50  0001 C CNN "LCSC"
+	2    2200 4200
+	1    0    0    -1
+$EndComp
+$Comp
+L 74xx:74HC00 U?
+U 1 1 60193F08
+P 1400 5100
+F 0 "U?" H 1400 5425 50  0000 C CNN
+F 1 "74HC00" H 1400 5334 50  0000 C CNN
+F 2 "Package_SO:TSSOP-14_4.4x5mm_P0.65mm" H 1400 5100 50  0001 C CNN
+F 3 "https://datasheet.lcsc.com/szlcsc/Texas-Instruments-TI-SN74HC00PWR_C6807.pdf" H 1400 5100 50  0001 C CNN
+F 4 "C6807" H 1400 5100 50  0001 C CNN "LCSC"
+	1    1400 5100
+	1    0    0    -1
+$EndComp
+$Comp
+L 74xx:74HC00 U?
+U 2 1 6019C24F
+P 2200 5100
+F 0 "U?" H 2200 5425 50  0000 C CNN
+F 1 "74HC00" H 2200 5334 50  0000 C CNN
+F 2 "Package_SO:TSSOP-14_4.4x5mm_P0.65mm" H 2200 5100 50  0001 C CNN
+F 3 "https://datasheet.lcsc.com/szlcsc/Texas-Instruments-TI-SN74HC00PWR_C6807.pdf" H 2200 5100 50  0001 C CNN
+F 4 "C6807" H 2200 5100 50  0001 C CNN "LCSC"
+	2    2200 5100
+	1    0    0    -1
+$EndComp
+$Comp
+L 74xx:74HC00 U?
+U 3 1 6019DAAA
+P 3000 5100
+F 0 "U?" H 3000 5425 50  0000 C CNN
+F 1 "74HC00" H 3000 5334 50  0000 C CNN
+F 2 "Package_SO:TSSOP-14_4.4x5mm_P0.65mm" H 3000 5100 50  0001 C CNN
+F 3 "https://datasheet.lcsc.com/szlcsc/Texas-Instruments-TI-SN74HC00PWR_C6807.pdf" H 3000 5100 50  0001 C CNN
+F 4 "C6807" H 3000 5100 50  0001 C CNN "LCSC"
+	3    3000 5100
+	1    0    0    -1
+$EndComp
+$Comp
+L 74xx:74HC00 U?
+U 5 1 601A0524
+P 4800 5650
+F 0 "U?" H 5030 5696 50  0000 L CNN
+F 1 "74HC00" H 5030 5605 50  0000 L CNN
+F 2 "Package_SO:TSSOP-14_4.4x5mm_P0.65mm" H 4800 5650 50  0001 C CNN
+F 3 "https://datasheet.lcsc.com/szlcsc/Texas-Instruments-TI-SN74HC00PWR_C6807.pdf" H 4800 5650 50  0001 C CNN
+F 4 "C6807" H 4800 5650 50  0001 C CNN "LCSC"
+	5    4800 5650
+	1    0    0    -1
+$EndComp
+$Comp
+L 74xx:74HC00 U?
+U 4 1 6019F25D
+P 3850 5100
+F 0 "U?" H 3850 5425 50  0000 C CNN
+F 1 "74HC00" H 3850 5334 50  0000 C CNN
+F 2 "Package_SO:TSSOP-14_4.4x5mm_P0.65mm" H 3850 5100 50  0001 C CNN
+F 3 "https://datasheet.lcsc.com/szlcsc/Texas-Instruments-TI-SN74HC00PWR_C6807.pdf" H 3850 5100 50  0001 C CNN
+F 4 "C6807" H 3850 5100 50  0001 C CNN "LCSC"
+	4    3850 5100
+	1    0    0    -1
+$EndComp
