File: PB170/output.sch (KiCad schematic (older format))
At the start: 0 parts

Commit message: ALU finished
Parts:
- added D? (x4): LED green, LEDs:LED_0603, symbol Device:LED
- added D?: LED red, LEDs:LED_0603, symbol Device:LED
- added D? (x2): LED yellow, LEDs:LED_0603, symbol Device:LED
- added R? (x6): 180R, Resistors_SMD:R_0603, symbol Device:R
- added R?: 220R, Resistors_SMD:R_0603, symbol Device:R
Connections:
- net IN_NF: now also D?.2 (A)
- net IN_OF: now also D?.2 (A)
- net IN_Y0: now also D?.2 (A)
- net IN_Y1: now also D?.2 (A)
- net IN_Y2: now also D?.2 (A)
- net IN_Y3: now also D?.2 (A)
- net IN_ZF: now also D?.2 (A)
- new net: D?.1 (K), R?.1 (x7)
- new net GND: R?.2, R?.2, R?.2, R?.2, R?.2, R?.2, R?.2
