File: PB170/PB170.kicad_pcb (KiCad board)
At the start: 4 copper layers, 96.5 x 71.1 mm, 39 parts, among them J2 USB_B_Micro, Q1 P-MOSFET-MLP_HS, Q2 BC817, SW1 SW_MEC_5E, SW2 SW_MEC_5E, SW3 SW_SPDT, U1 74HC00, U2 74HC08, U3 74HC4511D, U4 HEF4518BT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

Commit message: Fixed ovelapping parts.
Parts:
- moved RV1 72.7 mm to (61.6, 90.9)
- moved J2 46.2 mm to (79.1, 92.2)
- moved R11 34.2 mm to (78.7, 83.8)
- moved SW3 7.80 mm to (101.5, 32.3)
Routing:
- net Net-(J2-Pad3): track 3.47 -> 0.00 mm, vias 1 -> 0
- net Net-(J2-Pad2): track 3.11 -> 0.00 mm, vias 1 -> 0
