File: logic.sch (KiCad schematic (older format))
At the start: 10 parts

Commit message: Anotate alu
Parts:
- gave numbers to parts that had none: 2
Changed lines of the file:
@@
 IN_NOT_OR
 $Comp
-L PB170:74HC08 U?
+L PB170:74HC08 U8
 U 1 1 6012A899
 P 2300 1650
-F 0 "U?" H 2325 1917 50  0000 C CNN
+F 0 "U8" H 2325 1917 50  0000 C CNN
 F 1 "74HC08" H 2325 1826 50  0000 C CNN
 F 2 "Housings_SOIC:SOIC-14_3.9x8.7mm_Pitch1.27mm" H 2300 1650 50  0001 C CNN
@@
 $EndComp
 $Comp
-L PB170:74HC08 U?
+L PB170:74HC08 U8
 U 2 1 6012BE48
 P 2300 2050
-F 0 "U?" H 2325 2317 50  0000 C CNN
+F 0 "U8" H 2325 2317 50  0000 C CNN
 F 1 "74HC08" H 2325 2226 50  0000 C CNN
 F 2 "Housings_SOIC:SOIC-14_3.9x8.7mm_Pitch1.27mm" H 2300 2050 50  0001 C CNN
@@
 $EndComp
 $Comp
-L PB170:74HC08 U?
+L PB170:74HC08 U8
 U 3 1 6012CB7D
 P 2300 2450
-F 0 "U?" H 2325 2717 50  0000 C CNN
+F 0 "U8" H 2325 2717 50  0000 C CNN
 F 1 "74HC08" H 2325 2626 50  0000 C CNN
 F 2 "Housings_SOIC:SOIC-14_3.9x8.7mm_Pitch1.27mm" H 2300 2450 50  0001 C CNN
@@
 $EndComp
 $Comp
-L PB170:74HC08 U?
+L PB170:74HC08 U8
 U 4 1 6012D786
 P 2300 2850
-F 0 "U?" H 2325 3117 50  0000 C CNN
+F 0 "U8" H 2325 3117 50  0000 C CNN
 F 1 "74HC08" H 2325 3026 50  0000 C CNN
 F 2 "Housings_SOIC:SOIC-14_3.9x8.7mm_Pitch1.27mm" H 2300 2850 50  0001 C CNN
@@
 $EndComp
 $Comp
-L PB170:74HC08 U?
+L PB170:74HC08 U8
 U 5 1 6012E727
 P 3900 1650
-F 0 "U?" H 4130 1696 50  0000 L CNN
+F 0 "U8" H 4130 1696 50  0000 L CNN
 F 1 "74HC08" H 4130 1605 50  0000 L CNN
 F 2 "Housings_SOIC:SOIC-14_3.9x8.7mm_Pitch1.27mm" H 3900 1650 50  0001 C CNN
@@
 $EndComp
 $Comp
-L PB170:74HC32 U?
+L PB170:74HC32 U9
 U 1 1 60125BE5
 P 2350 3400
-F 0 "U?" H 2325 3675 50  0000 C CNN
+F 0 "U9" H 2325 3675 50  0000 C CNN
 F 1 "74HC32" H 2325 3584 50  0000 C CNN
 F 2 "Housings_SOIC:SOIC-14_3.9x8.7mm_Pitch1.27mm" H 1800 3600 50  0001 C CNN
@@
 $EndComp
 $Comp
-L PB170:74HC32 U?
+L PB170:74HC32 U9
 U 2 1 601271F6
 P 2350 3800
-F 0 "U?" H 2325 4075 50  0000 C CNN
+F 0 "U9" H 2325 4075 50  0000 C CNN
 F 1 "74HC32" H 2325 3984 50  0000 C CNN
 F 2 "Housings_SOIC:SOIC-14_3.9x8.7mm_Pitch1.27mm" H 1800 4000 50  0001 C CNN
@@
 $EndComp
 $Comp
-L PB170:74HC32 U?
+L PB170:74HC32 U9
 U 3 1 60128ABF
 P 2350 4200
-F 0 "U?" H 2325 4475 50  0000 C CNN
+F 0 "U9" H 2325 4475 50  0000 C CNN
 F 1 "74HC32" H 2325 4384 50  0000 C CNN
 F 2 "Housings_SOIC:SOIC-14_3.9x8.7mm_Pitch1.27mm" H 1800 4400 50  0001 C CNN
@@
 $EndComp
 $Comp
-L PB170:74HC32 U?
+L PB170:74HC32 U9
 U 4 1 6012A0B0
 P 2350 4600
-F 0 "U?" H 2325 4875 50  0000 C CNN
+F 0 "U9" H 2325 4875 50  0000 C CNN
 F 1 "74HC32" H 2325 4784 50  0000 C CNN
 F 2 "Housings_SOIC:SOIC-14_3.9x8.7mm_Pitch1.27mm" H 1800 4800 50  0001 C CNN
@@
 $EndComp
 $Comp
-L PB170:74HC32 U?
+L PB170:74HC32 U9
 U 5 1 6012B245
 P 3900 4100
-F 0 "U?" H 3778 4146 50  0000 L CNN
+F 0 "U9" H 3778 4146 50  0000 L CNN
 F 1 "74HC32" H 3778 4055 50  0000 L CNN
 F 2 "Housings_SOIC:SOIC-14_3.9x8.7mm_Pitch1.27mm" H 3350 4300 50  0001 C CNN

Commit message: fixed some footprints
Parts:
- U8, U9: footprint Housings_SOIC:SOIC-14_3.9x8.7mm_Pitch1.27mm -> Package_SO:SOIC-14_3.9x8.7mm_P1.27mm
Changed lines of the file:
@@
 F 0 "U8" H 2325 1917 50  0000 C CNN
 F 1 "74HC08" H 2325 1826 50  0000 C CNN
-F 2 "Housings_SOIC:SOIC-14_3.9x8.7mm_Pitch1.27mm" H 2300 1650 50  0001 C CNN
+F 2 "Package_SO:SOIC-14_3.9x8.7mm_P1.27mm" H 2300 1650 50  0001 C CNN
 F 3 "https://datasheet.lcsc.com/szlcsc/Nexperia-74HC08D-653_C5593.pdf" H 2300 1650 50  0001 C CNN
 F 4 "C5593" H 2300 1650 50  0001 C CNN "LCSC"
@@
 F 0 "U8" H 2325 2317 50  0000 C CNN
 F 1 "74HC08" H 2325 2226 50  0000 C CNN
-F 2 "Housings_SOIC:SOIC-14_3.9x8.7mm_Pitch1.27mm" H 2300 2050 50  0001 C CNN
+F 2 "Package_SO:SOIC-14_3.9x8.7mm_P1.27mm" H 2300 2050 50  0001 C CNN
 F 3 "https://datasheet.lcsc.com/szlcsc/Nexperia-74HC08D-653_C5593.pdf" H 2300 2050 50  0001 C CNN
 F 4 "C5593" H 2300 2050 50  0001 C CNN "LCSC"
@@
 F 0 "U8" H 2325 2717 50  0000 C CNN
 F 1 "74HC08" H 2325 2626 50  0000 C CNN
-F 2 "Housings_SOIC:SOIC-14_3.9x8.7mm_Pitch1.27mm" H 2300 2450 50  0001 C CNN
+F 2 "Package_SO:SOIC-14_3.9x8.7mm_P1.27mm" H 2300 2450 50  0001 C CNN
 F 3 "https://datasheet.lcsc.com/szlcsc/Nexperia-74HC08D-653_C5593.pdf" H 2300 2450 50  0001 C CNN
 F 4 "C5593" H 2300 2450 50  0001 C CNN "LCSC"
@@
 F 0 "U8" H 2325 3117 50  0000 C CNN
 F 1 "74HC08" H 2325 3026 50  0000 C CNN
-F 2 "Housings_SOIC:SOIC-14_3.9x8.7mm_Pitch1.27mm" H 2300 2850 50  0001 C CNN
+F 2 "Package_SO:SOIC-14_3.9x8.7mm_P1.27mm" H 2300 2850 50  0001 C CNN
 F 3 "https://datasheet.lcsc.com/szlcsc/Nexperia-74HC08D-653_C5593.pdf" H 2300 2850 50  0001 C CNN
 F 4 "C5593" H 2300 2850 50  0001 C CNN "LCSC"
@@
 F 0 "U8" H 4130 1696 50  0000 L CNN
 F 1 "74HC08" H 4130 1605 50  0000 L CNN
-F 2 "Housings_SOIC:SOIC-14_3.9x8.7mm_Pitch1.27mm" H 3900 1650 50  0001 C CNN
+F 2 "Package_SO:SOIC-14_3.9x8.7mm_P1.27mm" H 3900 1650 50  0001 C CNN
 F 3 "https://datasheet.lcsc.com/szlcsc/Nexperia-74HC08D-653_C5593.pdf" H 3900 1650 50  0001 C CNN
 F 4 "C5593" H 3900 1650 50  0001 C CNN "LCSC"
@@
 F 0 "U9" H 2325 3675 50  0000 C CNN
 F 1 "74HC32" H 2325 3584 50  0000 C CNN
-F 2 "Housings_SOIC:SOIC-14_3.9x8.7mm_Pitch1.27mm" H 1800 3600 50  0001 C CNN
+F 2 "Package_SO:SOIC-14_3.9x8.7mm_P1.27mm" H 1800 3600 50  0001 C CNN
 F 3 "https://datasheet.lcsc.com/szlcsc/Nexperia-74HC32D-653_C5632.pdf" H 1800 3600 50  0001 C CNN
 F 4 "C5632" H 2350 3400 50  0001 C CNN "LCSC"
@@
 F 0 "U9" H 2325 4075 50  0000 C CNN
 F 1 "74HC32" H 2325 3984 50  0000 C CNN
-F 2 "Housings_SOIC:SOIC-14_3.9x8.7mm_Pitch1.27mm" H 1800 4000 50  0001 C CNN
+F 2 "Package_SO:SOIC-14_3.9x8.7mm_P1.27mm" H 1800 4000 50  0001 C CNN
 F 3 "https://datasheet.lcsc.com/szlcsc/Nexperia-74HC32D-653_C5632.pdf" H 1800 4000 50  0001 C CNN
 F 4 "C5632" H 2350 3800 50  0001 C CNN "LCSC"
@@
 F 0 "U9" H 2325 4475 50  0000 C CNN
 F 1 "74HC32" H 2325 4384 50  0000 C CNN
-F 2 "Housings_SOIC:SOIC-14_3.9x8.7mm_Pitch1.27mm" H 1800 4400 50  0001 C CNN
+F 2 "Package_SO:SOIC-14_3.9x8.7mm_P1.27mm" H 1800 4400 50  0001 C CNN
 F 3 "https://datasheet.lcsc.com/szlcsc/Nexperia-74HC32D-653_C5632.pdf" H 1800 4400 50  0001 C CNN
 F 4 "C5632" H 2350 4200 50  0001 C CNN "LCSC"
@@
 F 0 "U9" H 2325 4875 50  0000 C CNN
 F 1 "74HC32" H 2325 4784 50  0000 C CNN
-F 2 "Housings_SOIC:SOIC-14_3.9x8.7mm_Pitch1.27mm" H 1800 4800 50  0001 C CNN
+F 2 "Package_SO:SOIC-14_3.9x8.7mm_P1.27mm" H 1800 4800 50  0001 C CNN
 F 3 "https://datasheet.lcsc.com/szlcsc/Nexperia-74HC32D-653_C5632.pdf" H 1800 4800 50  0001 C CNN
 F 4 "C5632" H 2350 4600 50  0001 C CNN "LCSC"
@@
 F 0 "U9" H 3778 4146 50  0000 L CNN
 F 1 "74HC32" H 3778 4055 50  0000 L CNN
-F 2 "Housings_SOIC:SOIC-14_3.9x8.7mm_Pitch1.27mm" H 3350 4300 50  0001 C CNN
+F 2 "Package_SO:SOIC-14_3.9x8.7mm_P1.27mm" H 3350 4300 50  0001 C CNN
 F 3 "https://datasheet.lcsc.com/szlcsc/Nexperia-74HC32D-653_C5632.pdf" H 3350 4300 50  0001 C CNN
 F 4 "C5632" H 3900 4100 50  0001 C CNN "LCSC"
