File: op-mux.sch (KiCad schematic (older format))
At the start: 15 parts

Commit message: Anotate alu
Parts:
- gave numbers to parts that had none: 3
Changed lines of the file:
@@
 IN_NOT_OP
 $Comp
-L PB170:74HC08 U?
+L PB170:74HC08 U13
 U 1 1 60130F9F
 P 1750 900
-AR Path="/600A4AF3/600D6CED/60130F9F" Ref="U?"  Part="1"
-AR Path="/600A4AF3/600D523C/6027A5F8/60130F9F" Ref="U?"  Part="1"
-F 0 "U?" H 1775 1167 50  0000 C CNN
+AR Path="/600A4AF3/600D6CED/60130F9F" Ref="U13"  Part="1"
+AR Path="/600A4AF3/600D523C/6027A5F8/60130F9F" Ref="U10"  Part="1"
+F 0 "U13" H 1775 1167 50  0000 C CNN
 F 1 "74HC08" H 1775 1076 50  0000 C CNN
 F 2 "Housings_SOIC:SOIC-14_3.9x8.7mm_Pitch1.27mm" H 1750 900 50  0001 C CNN
@@
 $EndComp
 $Comp
-L PB170:74HC08 U?
+L PB170:74HC08 U13
 U 2 1 60131E1E
 P 1750 1300
-AR Path="/600A4AF3/600D6CED/60131E1E" Ref="U?"  Part="2"
-AR Path="/600A4AF3/600D523C/6027A5F8/60131E1E" Ref="U?"  Part="2"
-F 0 "U?" H 1775 1567 50  0000 C CNN
+AR Path="/600A4AF3/600D6CED/60131E1E" Ref="U13"  Part="2"
+AR Path="/600A4AF3/600D523C/6027A5F8/60131E1E" Ref="U10"  Part="2"
+F 0 "U13" H 1775 1567 50  0000 C CNN
 F 1 "74HC08" H 1775 1476 50  0000 C CNN
 F 2 "Housings_SOIC:SOIC-14_3.9x8.7mm_Pitch1.27mm" H 1750 1300 50  0001 C CNN
@@
 $EndComp
 $Comp
-L PB170:74HC08 U?
+L PB170:74HC08 U13
 U 3 1 60132AD1
 P 1750 1700
-AR Path="/600A4AF3/600D6CED/60132AD1" Ref="U?"  Part="3"
-AR Path="/600A4AF3/600D523C/6027A5F8/60132AD1" Ref="U?"  Part="3"
-F 0 "U?" H 1775 1967 50  0000 C CNN
+AR Path="/600A4AF3/600D6CED/60132AD1" Ref="U13"  Part="3"
+AR Path="/600A4AF3/600D523C/6027A5F8/60132AD1" Ref="U10"  Part="3"
+F 0 "U13" H 1775 1967 50  0000 C CNN
 F 1 "74HC08" H 1775 1876 50  0000 C CNN
 F 2 "Housings_SOIC:SOIC-14_3.9x8.7mm_Pitch1.27mm" H 1750 1700 50  0001 C CNN
@@
 $EndComp
 $Comp
-L PB170:74HC08 U?
+L PB170:74HC08 U13
 U 4 1 601333C0
 P 1750 2100
-AR Path="/600A4AF3/600D6CED/601333C0" Ref="U?"  Part="4"
-AR Path="/600A4AF3/600D523C/6027A5F8/601333C0" Ref="U?"  Part="4"
-F 0 "U?" H 1775 2367 50  0000 C CNN
+AR Path="/600A4AF3/600D6CED/601333C0" Ref="U13"  Part="4"
+AR Path="/600A4AF3/600D523C/6027A5F8/601333C0" Ref="U10"  Part="4"
+F 0 "U13" H 1775 2367 50  0000 C CNN
 F 1 "74HC08" H 1775 2276 50  0000 C CNN
 F 2 "Housings_SOIC:SOIC-14_3.9x8.7mm_Pitch1.27mm" H 1750 2100 50  0001 C CNN
@@
 $EndComp
 $Comp
-L PB170:74HC08 U?
+L PB170:74HC08 U14
 U 5 1 60133CF5
 P 3450 3950
-AR Path="/600A4AF3/600D6CED/60133CF5" Ref="U?"  Part="5"
-AR Path="/600A4AF3/600D523C/6027A5F8/60133CF5" Ref="U?"  Part="5"
-F 0 "U?" V 3083 3950 50  0000 C CNN
+AR Path="/600A4AF3/600D6CED/60133CF5" Ref="U14"  Part="5"
+AR Path="/600A4AF3/600D523C/6027A5F8/60133CF5" Ref="U11"  Part="5"
+F 0 "U14" V 3083 3950 50  0000 C CNN
 F 1 "74HC08" V 3174 3950 50  0000 C CNN
 F 2 "Housings_SOIC:SOIC-14_3.9x8.7mm_Pitch1.27mm" H 3450 3950 50  0001 C CNN
@@
 $EndComp
 $Comp
-L PB170:74HC08 U?
+L PB170:74HC08 U14
 U 1 1 601447C3
 P 1750 2700
-AR Path="/600A4AF3/600D6CED/601447C3" Ref="U?"  Part="1"
-AR Path="/600A4AF3/600D523C/6027A5F8/601447C3" Ref="U?"  Part="1"
-F 0 "U?" H 1775 2967 50  0000 C CNN
+AR Path="/600A4AF3/600D6CED/601447C3" Ref="U14"  Part="1"
+AR Path="/600A4AF3/600D523C/6027A5F8/601447C3" Ref="U11"  Part="1"
+F 0 "U14" H 1775 2967 50  0000 C CNN
 F 1 "74HC08" H 1775 2876 50  0000 C CNN
 F 2 "Housings_SOIC:SOIC-14_3.9x8.7mm_Pitch1.27mm" H 1750 2700 50  0001 C CNN
@@
 $EndComp
 $Comp
-L PB170:74HC08 U?
+L PB170:74HC08 U14
 U 2 1 601447CA
 P 1750 3100
-AR Path="/600A4AF3/600D6CED/601447CA" Ref="U?"  Part="2"
-AR Path="/600A4AF3/600D523C/6027A5F8/601447CA" Ref="U?"  Part="2"
-F 0 "U?" H 1775 3367 50  0000 C CNN
+AR Path="/600A4AF3/600D6CED/601447CA" Ref="U14"  Part="2"
+AR Path="/600A4AF3/600D523C/6027A5F8/601447CA" Ref="U11"  Part="2"
+F 0 "U14" H 1775 3367 50  0000 C CNN
 F 1 "74HC08" H 1775 3276 50  0000 C CNN
 F 2 "Housings_SOIC:SOIC-14_3.9x8.7mm_Pitch1.27mm" H 1750 3100 50  0001 C CNN
@@
 $EndComp
 $Comp
-L PB170:74HC08 U?
+L PB170:74HC08 U14
 U 3 1 601447D1
 P 1750 3500
-AR Path="/600A4AF3/600D6CED/601447D1" Ref="U?"  Part="3"
-AR Path="/600A4AF3/600D523C/6027A5F8/601447D1" Ref="U?"  Part="3"
-F 0 "U?" H 1775 3767 50  0000 C CNN
+AR Path="/600A4AF3/600D6CED/601447D1" Ref="U14"  Part="3"
+AR Path="/600A4AF3/600D523C/6027A5F8/601447D1" Ref="U11"  Part="3"
+F 0 "U14" H 1775 3767 50  0000 C CNN
 F 1 "74HC08" H 1775 3676 50  0000 C CNN
 F 2 "Housings_SOIC:SOIC-14_3.9x8.7mm_Pitch1.27mm" H 1750 3500 50  0001 C CNN
@@
 $EndComp
 $Comp
-L PB170:74HC08 U?
+L PB170:74HC08 U14
 U 4 1 601447D8
 P 1750 3900
-AR Path="/600A4AF3/600D6CED/601447D8" Ref="U?"  Part="4"
-AR Path="/600A4AF3/600D523C/6027A5F8/601447D8" Ref="U?"  Part="4"
-F 0 "U?" H 1775 4167 50  0000 C CNN
+AR Path="/600A4AF3/600D6CED/601447D8" Ref="U14"  Part="4"
+AR Path="/600A4AF3/600D523C/6027A5F8/601447D8" Ref="U11"  Part="4"
+F 0 "U14" H 1775 4167 50  0000 C CNN
 F 1 "74HC08" H 1775 4076 50  0000 C CNN
 F 2 "Housings_SOIC:SOIC-14_3.9x8.7mm_Pitch1.27mm" H 1750 3900 50  0001 C CNN
@@
 $EndComp
 $Comp
-L PB170:74HC08 U?
+L PB170:74HC08 U13
 U 5 1 601447DF
 P 3450 3250
-AR Path="/600A4AF3/600D6CED/601447DF" Ref="U?"  Part="5"
-AR Path="/600A4AF3/600D523C/6027A5F8/601447DF" Ref="U?"  Part="5"
-F 0 "U?" V 3083 3250 50  0000 C CNN
+AR Path="/600A4AF3/600D6CED/601447DF" Ref="U13"  Part="5"
+AR Path="/600A4AF3/600D523C/6027A5F8/601447DF" Ref="U10"  Part="5"
+F 0 "U13" V 3083 3250 50  0000 C CNN
 F 1 "74HC08" V 3174 3250 50  0000 C CNN
 F 2 "Housings_SOIC:SOIC-14_3.9x8.7mm_Pitch1.27mm" H 3450 3250 50  0001 C CNN
@@
 	1250 2650 1000 2650
 $Comp
-L PB170:74HC32 U?
+L PB170:74HC32 U15
 U 1 1 6021F5C2
 P 3000 950
-AR Path="/600A4AF3/600D6CED/6021F5C2" Ref="U?"  Part="1"
-AR Path="/600A4AF3/600D523C/6027A5F8/6021F5C2" Ref="U?"  Part="1"
-F 0 "U?" H 2975 1225 50  0000 C CNN
+AR Path="/600A4AF3/600D6CED/6021F5C2" Ref="U15"  Part="1"
+AR Path="/600A4AF3/600D523C/6027A5F8/6021F5C2" Ref="U12"  Part="1"
+F 0 "U15" H 2975 1225 50  0000 C CNN
 F 1 "74HC32" H 2975 1134 50  0000 C CNN
 F 2 "Housings_SOIC:SOIC-14_3.9x8.7mm_Pitch1.27mm" H 2450 1150 50  0001 C CNN
@@
 $EndComp
 $Comp
-L PB170:74HC32 U?
+L PB170:74HC32 U15
 U 2 1 60221D93
 P 3000 1350
-AR Path="/600A4AF3/600D6CED/60221D93" Ref="U?"  Part="2"
-AR Path="/600A4AF3/600D523C/6027A5F8/60221D93" Ref="U?"  Part="2"
-F 0 "U?" H 2975 1625 50  0000 C CNN
+AR Path="/600A4AF3/600D6CED/60221D93" Ref="U15"  Part="2"
+AR Path="/600A4AF3/600D523C/6027A5F8/60221D93" Ref="U12"  Part="2"
+F 0 "U15" H 2975 1625 50  0000 C CNN
 F 1 "74HC32" H 2975 1534 50  0000 C CNN
 F 2 "Housings_SOIC:SOIC-14_3.9x8.7mm_Pitch1.27mm" H 2450 1550 50  0001 C CNN
@@
 $EndComp
 $Comp
-L PB170:74HC32 U?
+L PB170:74HC32 U15
 U 3 1 6022339E
 P 3000 1750
-AR Path="/600A4AF3/600D6CED/6022339E" Ref="U?"  Part="3"
-AR Path="/600A4AF3/600D523C/6027A5F8/6022339E" Ref="U?"  Part="3"
-F 0 "U?" H 2975 2025 50  0000 C CNN
+AR Path="/600A4AF3/600D6CED/6022339E" Ref="U15"  Part="3"
+AR Path="/600A4AF3/600D523C/6027A5F8/6022339E" Ref="U12"  Part="3"
+F 0 "U15" H 2975 2025 50  0000 C CNN
 F 1 "74HC32" H 2975 1934 50  0000 C CNN
 F 2 "Housings_SOIC:SOIC-14_3.9x8.7mm_Pitch1.27mm" H 2450 1950 50  0001 C CNN
@@
 $EndComp
 $Comp
-L PB170:74HC32 U?
+L PB170:74HC32 U15
 U 4 1 60224D65
 P 3000 2150
-AR Path="/600A4AF3/600D6CED/60224D65" Ref="U?"  Part="4"
-AR Path="/600A4AF3/600D523C/6027A5F8/60224D65" Ref="U?"  Part="4"
-F 0 "U?" H 2975 2425 50  0000 C CNN
+AR Path="/600A4AF3/600D6CED/60224D65" Ref="U15"  Part="4"
+AR Path="/600A4AF3/600D523C/6027A5F8/60224D65" Ref="U12"  Part="4"
+F 0 "U15" H 2975 2425 50  0000 C CNN
 F 1 "74HC32" H 2975 2334 50  0000 C CNN
 F 2 "Housings_SOIC:SOIC-14_3.9x8.7mm_Pitch1.27mm" H 2450 2350 50  0001 C CNN
@@
 $EndComp
 $Comp
-L PB170:74HC32 U?
+L PB170:74HC32 U15
 U 5 1 60225F80
 P 3450 2950
-AR Path="/600A4AF3/600D6CED/60225F80" Ref="U?"  Part="5"
-AR Path="/600A4AF3/600D523C/6027A5F8/60225F80" Ref="U?"  Part="5"
-F 0 "U?" V 2835 2950 50  0000 C CNN
+AR Path="/600A4AF3/600D6CED/60225F80" Ref="U15"  Part="5"
+AR Path="/600A4AF3/600D523C/6027A5F8/60225F80" Ref="U12"  Part="5"
+F 0 "U15" V 2835 2950 50  0000 C CNN
 F 1 "74HC32" V 2926 2950 50  0000 C CNN
 F 2 "Housings_SOIC:SOIC-14_3.9x8.7mm_Pitch1.27mm" H 2900 3150 50  0001 C CNN

Commit message: fixed some footprints
Parts:
- U13, U14, U15: footprint Housings_SOIC:SOIC-14_3.9x8.7mm_Pitch1.27mm -> Package_SO:SOIC-14_3.9x8.7mm_P1.27mm
Changed lines of the file:
@@
 F 0 "U13" H 1775 1167 50  0000 C CNN
 F 1 "74HC08" H 1775 1076 50  0000 C CNN
-F 2 "Housings_SOIC:SOIC-14_3.9x8.7mm_Pitch1.27mm" H 1750 900 50  0001 C CNN
+F 2 "Package_SO:SOIC-14_3.9x8.7mm_P1.27mm" H 1750 900 50  0001 C CNN
 F 3 "https://datasheet.lcsc.com/szlcsc/Nexperia-74HC08D-653_C5593.pdf" H 1750 900 50  0001 C CNN
 F 4 "C5593" H 1750 900 50  0001 C CNN "LCSC"
@@
 F 0 "U13" H 1775 1567 50  0000 C CNN
 F 1 "74HC08" H 1775 1476 50  0000 C CNN
-F 2 "Housings_SOIC:SOIC-14_3.9x8.7mm_Pitch1.27mm" H 1750 1300 50  0001 C CNN
+F 2 "Package_SO:SOIC-14_3.9x8.7mm_P1.27mm" H 1750 1300 50  0001 C CNN
 F 3 "https://datasheet.lcsc.com/szlcsc/Nexperia-74HC08D-653_C5593.pdf" H 1750 1300 50  0001 C CNN
 F 4 "C5593" H 1750 1300 50  0001 C CNN "LCSC"
@@
 F 0 "U13" H 1775 1967 50  0000 C CNN
 F 1 "74HC08" H 1775 1876 50  0000 C CNN
-F 2 "Housings_SOIC:SOIC-14_3.9x8.7mm_Pitch1.27mm" H 1750 1700 50  0001 C CNN
+F 2 "Package_SO:SOIC-14_3.9x8.7mm_P1.27mm" H 1750 1700 50  0001 C CNN
 F 3 "https://datasheet.lcsc.com/szlcsc/Nexperia-74HC08D-653_C5593.pdf" H 1750 1700 50  0001 C CNN
 F 4 "C5593" H 1750 1700 50  0001 C CNN "LCSC"
@@
 F 0 "U13" H 1775 2367 50  0000 C CNN
 F 1 "74HC08" H 1775 2276 50  0000 C CNN
-F 2 "Housings_SOIC:SOIC-14_3.9x8.7mm_Pitch1.27mm" H 1750 2100 50  0001 C CNN
+F 2 "Package_SO:SOIC-14_3.9x8.7mm_P1.27mm" H 1750 2100 50  0001 C CNN
 F 3 "https://datasheet.lcsc.com/szlcsc/Nexperia-74HC08D-653_C5593.pdf" H 1750 2100 50  0001 C CNN
 F 4 "C5593" H 1750 2100 50  0001 C CNN "LCSC"
@@
 F 0 "U14" V 3083 3950 50  0000 C CNN
 F 1 "74HC08" V 3174 3950 50  0000 C CNN
-F 2 "Housings_SOIC:SOIC-14_3.9x8.7mm_Pitch1.27mm" H 3450 3950 50  0001 C CNN
+F 2 "Package_SO:SOIC-14_3.9x8.7mm_P1.27mm" H 3450 3950 50  0001 C CNN
 F 3 "https://datasheet.lcsc.com/szlcsc/Nexperia-74HC08D-653_C5593.pdf" H 3450 3950 50  0001 C CNN
 F 4 "C5593" H 3450 3950 50  0001 C CNN "LCSC"
@@
 F 0 "U14" H 1775 2967 50  0000 C CNN
 F 1 "74HC08" H 1775 2876 50  0000 C CNN
-F 2 "Housings_SOIC:SOIC-14_3.9x8.7mm_Pitch1.27mm" H 1750 2700 50  0001 C CNN
+F 2 "Package_SO:SOIC-14_3.9x8.7mm_P1.27mm" H 1750 2700 50  0001 C CNN
 F 3 "https://datasheet.lcsc.com/szlcsc/Nexperia-74HC08D-653_C5593.pdf" H 1750 2700 50  0001 C CNN
 F 4 "C5593" H 1750 2700 50  0001 C CNN "LCSC"
@@
 F 0 "U14" H 1775 3367 50  0000 C CNN
 F 1 "74HC08" H 1775 3276 50  0000 C CNN
-F 2 "Housings_SOIC:SOIC-14_3.9x8.7mm_Pitch1.27mm" H 1750 3100 50  0001 C CNN
+F 2 "Package_SO:SOIC-14_3.9x8.7mm_P1.27mm" H 1750 3100 50  0001 C CNN
 F 3 "https://datasheet.lcsc.com/szlcsc/Nexperia-74HC08D-653_C5593.pdf" H 1750 3100 50  0001 C CNN
 F 4 "C5593" H 1750 3100 50  0001 C CNN "LCSC"
@@
 F 0 "U14" H 1775 3767 50  0000 C CNN
 F 1 "74HC08" H 1775 3676 50  0000 C CNN
-F 2 "Housings_SOIC:SOIC-14_3.9x8.7mm_Pitch1.27mm" H 1750 3500 50  0001 C CNN
+F 2 "Package_SO:SOIC-14_3.9x8.7mm_P1.27mm" H 1750 3500 50  0001 C CNN
 F 3 "https://datasheet.lcsc.com/szlcsc/Nexperia-74HC08D-653_C5593.pdf" H 1750 3500 50  0001 C CNN
 F 4 "C5593" H 1750 3500 50  0001 C CNN "LCSC"
@@
 F 0 "U14" H 1775 4167 50  0000 C CNN
 F 1 "74HC08" H 1775 4076 50  0000 C CNN
-F 2 "Housings_SOIC:SOIC-14_3.9x8.7mm_Pitch1.27mm" H 1750 3900 50  0001 C CNN
+F 2 "Package_SO:SOIC-14_3.9x8.7mm_P1.27mm" H 1750 3900 50  0001 C CNN
 F 3 "https://datasheet.lcsc.com/szlcsc/Nexperia-74HC08D-653_C5593.pdf" H 1750 3900 50  0001 C CNN
 F 4 "C5593" H 1750 3900 50  0001 C CNN "LCSC"
@@
 F 0 "U13" V 3083 3250 50  0000 C CNN
 F 1 "74HC08" V 3174 3250 50  0000 C CNN
-F 2 "Housings_SOIC:SOIC-14_3.9x8.7mm_Pitch1.27mm" H 3450 3250 50  0001 C CNN
+F 2 "Package_SO:SOIC-14_3.9x8.7mm_P1.27mm" H 3450 3250 50  0001 C CNN
 F 3 "https://datasheet.lcsc.com/szlcsc/Nexperia-74HC08D-653_C5593.pdf" H 3450 3250 50  0001 C CNN
 F 4 "C5593" H 3450 3250 50  0001 C CNN "LCSC"
@@
 F 0 "U15" H 2975 1225 50  0000 C CNN
 F 1 "74HC32" H 2975 1134 50  0000 C CNN
-F 2 "Housings_SOIC:SOIC-14_3.9x8.7mm_Pitch1.27mm" H 2450 1150 50  0001 C CNN
+F 2 "Package_SO:SOIC-14_3.9x8.7mm_P1.27mm" H 2450 1150 50  0001 C CNN
 F 3 "https://datasheet.lcsc.com/szlcsc/Nexperia-74HC32D-653_C5632.pdf" H 2450 1150 50  0001 C CNN
 F 4 "C5632" H 3000 950 50  0001 C CNN "LCSC"
@@
 F 0 "U15" H 2975 1625 50  0000 C CNN
 F 1 "74HC32" H 2975 1534 50  0000 C CNN
-F 2 "Housings_SOIC:SOIC-14_3.9x8.7mm_Pitch1.27mm" H 2450 1550 50  0001 C CNN
+F 2 "Package_SO:SOIC-14_3.9x8.7mm_P1.27mm" H 2450 1550 50  0001 C CNN
 F 3 "https://datasheet.lcsc.com/szlcsc/Nexperia-74HC32D-653_C5632.pdf" H 2450 1550 50  0001 C CNN
 F 4 "C5632" H 3000 1350 50  0001 C CNN "LCSC"
@@
 F 0 "U15" H 2975 2025 50  0000 C CNN
 F 1 "74HC32" H 2975 1934 50  0000 C CNN
-F 2 "Housings_SOIC:SOIC-14_3.9x8.7mm_Pitch1.27mm" H 2450 1950 50  0001 C CNN
+F 2 "Package_SO:SOIC-14_3.9x8.7mm_P1.27mm" H 2450 1950 50  0001 C CNN
 F 3 "https://datasheet.lcsc.com/szlcsc/Nexperia-74HC32D-653_C5632.pdf" H 2450 1950 50  0001 C CNN
 F 4 "C5632" H 3000 1750 50  0001 C CNN "LCSC"
@@
 F 0 "U15" H 2975 2425 50  0000 C CNN
 F 1 "74HC32" H 2975 2334 50  0000 C CNN
-F 2 "Housings_SOIC:SOIC-14_3.9x8.7mm_Pitch1.27mm" H 2450 2350 50  0001 C CNN
+F 2 "Package_SO:SOIC-14_3.9x8.7mm_P1.27mm" H 2450 2350 50  0001 C CNN
 F 3 "https://datasheet.lcsc.com/szlcsc/Nexperia-74HC32D-653_C5632.pdf" H 2450 2350 50  0001 C CNN
 F 4 "C5632" H 3000 2150 50  0001 C CNN "LCSC"
@@
 F 0 "U15" V 2835 2950 50  0000 C CNN
 F 1 "74HC32" V 2926 2950 50  0000 C CNN
-F 2 "Housings_SOIC:SOIC-14_3.9x8.7mm_Pitch1.27mm" H 2900 3150 50  0001 C CNN
+F 2 "Package_SO:SOIC-14_3.9x8.7mm_P1.27mm" H 2900 3150 50  0001 C CNN
 F 3 "https://datasheet.lcsc.com/szlcsc/Nexperia-74HC32D-653_C5632.pdf" H 2900 3150 50  0001 C CNN
 F 4 "C5632" H 3450 2950 50  0001 C CNN "LCSC"
@@
 AR Path="/600A4AF3/600D523C/6027A5F8/603A236A" Ref="#PWR0151"  Part="1"
 AR Path="/600A4AF3/600D6CED/603A236A" Ref="#PWR0141"  Part="1"
-F 0 "#PWR0141" H 3950 3800 50  0001 C CNN
+F 0 "#PWR0151" H 3950 3800 50  0001 C CNN
 F 1 "+5V" V 3965 4078 50  0000 L CNN
 F 2 "" H 3950 3950 50  0001 C CNN
@@
 AR Path="/600A4AF3/600D523C/6027A5F8/603A3AC8" Ref="#PWR0152"  Part="1"
 AR Path="/600A4AF3/600D6CED/603A3AC8" Ref="#PWR0142"  Part="1"
-F 0 "#PWR0142" H 3950 3100 50  0001 C CNN
+F 0 "#PWR0152" H 3950 3100 50  0001 C CNN
 F 1 "+5V" V 3965 3378 50  0000 L CNN
 F 2 "" H 3950 3250 50  0001 C CNN
@@
 AR Path="/600A4AF3/600D523C/6027A5F8/603A762B" Ref="#PWR0153"  Part="1"
 AR Path="/600A4AF3/600D6CED/603A762B" Ref="#PWR0143"  Part="1"
-F 0 "#PWR0143" H 3800 2500 50  0001 C CNN
+F 0 "#PWR0153" H 3800 2500 50  0001 C CNN
 F 1 "+5V" V 3815 2778 50  0000 L CNN
 F 2 "" H 3800 2650 50  0001 C CNN
@@
 AR Path="/600A4AF3/600D523C/6027A5F8/603CB24C" Ref="#PWR0154"  Part="1"
 AR Path="/600A4AF3/600D6CED/603CB24C" Ref="#PWR0144"  Part="1"
-F 0 "#PWR0144" H 2950 3700 50  0001 C CNN
+F 0 "#PWR0154" H 2950 3700 50  0001 C CNN
 F 1 "GND" V 2955 3822 50  0000 R CNN
 F 2 "" H 2950 3950 50  0001 C CNN
@@
 AR Path="/600A4AF3/600D523C/6027A5F8/603CCA4E" Ref="#PWR0155"  Part="1"
 AR Path="/600A4AF3/600D6CED/603CCA4E" Ref="#PWR0145"  Part="1"
-F 0 "#PWR0145" H 2950 3000 50  0001 C CNN
+F 0 "#PWR0155" H 2950 3000 50  0001 C CNN
 F 1 "GND" V 2955 3122 50  0000 R CNN
 F 2 "" H 2950 3250 50  0001 C CNN
@@
 AR Path="/600A4AF3/600D523C/6027A5F8/603CE342" Ref="#PWR0156"  Part="1"
 AR Path="/600A4AF3/600D6CED/603CE342" Ref="#PWR0146"  Part="1"
-F 0 "#PWR0146" H 3100 2400 50  0001 C CNN
+F 0 "#PWR0156" H 3100 2400 50  0001 C CNN
 F 1 "GND" V 3105 2522 50  0000 R CNN
 F 2 "" H 3100 2650 50  0001 C CNN
